Commit message: jtc: Add joint limits spec to rrbot test robot

File: joint_trajectory_controller/test/rrbot.xacro (robot description, xacro)
@@ -52,4 +52,5 @@
     <axis xyz="0 1 0"/>
     <dynamics damping="0.7"/>
+    <limit effort="20" velocity="${2*PI}" />
   </joint>
   <!-- Middle Link -->
@@ -83,4 +84,5 @@
     <axis xyz="0 1 0"/>
     <dynamics damping="0.7"/>
+    <limit effort="20" velocity="${2*PI}" />
   </joint>
   <!-- Top Link -->
