Commit message: Start controllers before test

File: effort_controllers/test/simple_bot.xacro (robot description, xacro)
@@ -14,5 +14,5 @@
     <axis xyz="0 0 1"/>
     <origin xyz="0 0 1"/>
-    <limit lower="-6.3" upper="6.3" effort="${1e6}" velocity="${1e4}"/>
+    <limit lower="-6.3" upper="6.3" effort="10" velocity="2"/>
   </joint>
   <transmission name="transimssion">
